Commit message: 2nd submit

File: src/my_robot/urdf/my_robot.xacro (robot description, xacro)
@@ -163,5 +163,5 @@
       <origin xyz="0 0 0" rpy="0 0 0"/>
       <geometry>
-    <box size="0.1 0.1 0.1"/>
+    	<box size="0.1 0.1 0.1"/>
       </geometry>
     </collision>
@@ -178,3 +178,9 @@
     </inertial>
   </link>
+  <joint name="hokuyo" type="fixed">
+   <axis xyz="0 1 0" rpy="0 0 0" />
+    <origin xyz="0.15 0 0.1" rpy="0 0 0"/>
+    <parent link="chassis" />
+    <child link="hokuyo" />
+  </joint>
 </robot>

Commit message: fix world

File: src/my_robot/urdf/my_robot.xacro (robot description, xacro)
@@ -184,3 +184,9 @@
     <child link="hokuyo" />
   </joint>
+  <gazebo reference="left_wheel">
+    <material>Gazebo/Blue</material>
+  </gazebo>
+  <gazebo reference="right_wheel">
+    <material>Gazebo/Red</material>
+  </gazebo>
 </robot>

Commit message: 3rd submit

File: src/my_robot/urdf/my_robot.xacro (robot description, xacro)
@@ -190,3 +190,6 @@
     <material>Gazebo/Red</material>
   </gazebo>
+  <gazebo reference="camera">
+    <material>Gazebo/Yellow</material>
+  </gazebo>
 </robot>

Commit message: submit 4th

File: src/my_robot/urdf/my_robot.xacro (robot description, xacro)
@@ -152,10 +152,4 @@
     <child link="camera"/>
   </joint>
-  <joint name="hokuyo_joint" type="fixed">
-    <axis xyz="0 1 0" />
-    <origin xyz=".15 0 .1" rpy="0 0 0"/>
-    <parent link="chassis"/>
-    <child link="hokuyo"/>
-  </joint>
   <!-- Hokuyo Laser -->
   <link name="hokuyo">

Commit message: modify my_robot

File: src/my_robot/urdf/my_robot.xacro (robot description, xacro)
@@ -179,8 +179,11 @@
   </joint>
   <gazebo reference="left_wheel">
-    <material>Gazebo/Blue</material>
+    <material>Gazebo/Red</material>
   </gazebo>
   <gazebo reference="right_wheel">
     <material>Gazebo/Red</material>
+  </gazebo>
+  <gazebo reference="chassis">
+    <material>Gazebo/Green</material>
   </gazebo>
   <gazebo reference="camera">

Commit message: before submit

File: src/my_robot/urdf/my_robot.xacro (robot description, xacro)
@@ -152,10 +152,4 @@
     <child link="camera"/>
   </joint>
-  <joint name="hokuyo_joint" type="fixed">
-    <axis xyz="0 1 0" />
-    <origin xyz=".15 0 .1" rpy="0 0 0"/>
-    <parent link="chassis"/>
-    <child link="hokuyo"/>
-  </joint>
   <!-- Hokuyo Laser -->
   <link name="hokuyo">
@@ -185,8 +179,11 @@
   </joint>
   <gazebo reference="left_wheel">
-    <material>Gazebo/Blue</material>
+    <material>Gazebo/Red</material>
   </gazebo>
   <gazebo reference="right_wheel">
     <material>Gazebo/Red</material>
+  </gazebo>
+  <gazebo reference="chassis">
+    <material>Gazebo/Green</material>
   </gazebo>
   <gazebo reference="camera">

Commit message: 1st commit

File: src/my_robot/urdf/my_robot.xacro (robot description, xacro)
@@ -145,5 +145,5 @@
       <inertia ixx="1e-6" ixy="0" ixz="0" iyy="1e-6" iyz="0" izz="1e-6" />
     </inertial>
-  </link>
+</link>
   <joint name="camera_joint" type="fixed">
     <axis xyz="0 1 0" />
@@ -151,4 +151,10 @@
     <parent link="chassis"/>
     <child link="camera"/>
+  </joint>
+  <link name="camera_rgbd_frame"></link>
+  <joint name="camera_rgbd_joint" type="fixed">
+    <origin xyz="0 0 0" rpy="-${pi/2} 0 -${pi/2}"/>
+    <parent link="camera"/>
+    <child link="camera_rgbd_frame"/>
   </joint>
   <!-- Hokuyo Laser -->
